Commit message: Reorganized packages and prepared names for release.
Signed-off-by: Ralph Lange (CR/AEE1) <ralph.lange@de.bosch.com>

File: micro-ros_kobuki-demo_kobuki-description/urdf/kobuki.urdf (robot description, URDF)
Before this commit: robot kobuki, 10 links, 9 joints
Links:
- link base_link: geometry collision cylinder length=0.10938 radius=0.178; visual mesh filename=package://micro-ros_kobuki-demo_kobuki-description/meshes/m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
- link wheel_left_link: geometry collision cylinder length=0.0206 radius=0.0352; visual mesh filename=package://micro-ros_kobuki-demo_kobuki-description/meshes/w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
- link wheel_right_link: geometry collision cylinder length=0.0206 radius=0.0350; visual mesh filename=package://micro-ros_kobuki-demo_kobuki-description/meshes/w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

Commit message: Harmonized names of packages, etc.
Signed-off-by: Ralph Lange (CR/AEE1) <ralph.lange@de.bosch.com>

File: micro-ros_kobuki-demo_kobuki-description/urdf/kobuki.urdf (robot description, URDF)
Before this commit: robot kobuki, 10 links, 9 joints
Links:
- link base_link: geometry collision cylinder length=0.10938 radius=0.178; visual mesh filename=package://micro-ros_kobuki_demo_robot-description/meshes/ma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
- link wheel_left_link: geometry collision cylinder length=0.0206 radius=0.0352; visual mesh filename=package://micro-ros_kobuki_demo_robot-description/meshes/wh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
- link wheel_right_link: geometry collision cylinder length=0.0206 radius=0.0350; visual mesh filename=package://micro-ros_kobuki_demo_robot-description/meshes/wh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
