Commit message: Improved URDF model.
Signed-off-by: Ralph Lange (CR/AEE1) <ralph.lange@de.bosch.com>

File: micro-ros_kobuki_demo_robot-description/urdf/kobuki.urdf (robot description, URDF)
Before this commit: robot kobuki, 10 links, 9 joints
Links:
- added link olimex_board; visual mesh filename=package://micro-ros_kobuki_demo_robot-description/meshes/ol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 scale=0.5 0.5 0.5
Joints:
- added joint olimex_board_joint: type fixed, parent base_link, child olimex_board, origin xyz=-0.03 0.071 0.09 rpy=0 0 0

Commit message: Scaled Olimex board model to correct size.
Signed-off-by: Ralph Lange <ralph.lange@de.bosch.com>

File: micro-ros_kobuki_demo_robot-description/urdf/kobuki.urdf (robot description, URDF)
Before this commit: robot kobuki, 11 links, 10 joints
Links:
- link olimex_board: geometry visual mesh filename=package://micro-ros_kobuki_demo_robot-description/meshes/ol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
