Commit message: Path fix in 3D models

File: micro-ros_crazyflie_demo_robot-description/urdf/crazyflie2.xacro (robot description, xacro)
@@ -14,5 +14,5 @@
       <origin xyz="0 0 0" rpy="0 0 0" />
       <geometry>
-        <mesh filename="package://crazyflie_description/meshes/crazyflie2.dae"/>
+        <mesh filename="package://micro-ros_crazyflie_demo_robot-description/meshes/crazyflie2.dae"/>
       </geometry>
     </visual>

File: micro-ros_crazyflie_demo_robot-description/urdf/crazyflie2_attitude.xacro (robot description, xacro)
@@ -14,5 +14,5 @@
       <origin xyz="0 0 0" rpy="0 0 0" />
       <geometry>
-        <mesh filename="package://crazyflie_description/meshes/crazyflie2.dae"/>
+        <mesh filename="package://micro-ros_crazyflie_demo_robot-description/meshes/crazyflie2.dae"/>
       </geometry>
     </visual>
